Commit message: comment out wobj_reference frame and change rviz setup

File: gluebot_support/urdf/gluebot.xacro (robot description, xacro)
@@ -15,4 +15,10 @@
   />
   <link name="world" />
+  <link name="camera_frame"/>
+  <joint name="world_to_camera" type="fixed">
+    <parent link="world"/>
+    <child link="camera_frame"/>
+    <origin xyz="-0.25 -0.5 1.25" rpy="0 3.14159 0"/>
+  </joint>
   <link name="table">
     <visual>
@@ -29,6 +35,6 @@
 		  </collision>
   </link>
-  <link name="wobj_reference"/>
-  <link name="wobj">
+  <!-- <link name="wobj_reference"/> -->
+  <!-- <link name="wobj">
     <visual>
       <geometry>
@@ -43,5 +49,5 @@
 			  <origin rpy="0 0 0" xyz="0 0 0"/>
 		</collision>
-  </link>
+  </link> -->
   <link name="glue_gun">
     <visual>
@@ -69,14 +75,14 @@
     <origin xyz="0.0 0.0 0.0" rpy="0.0 0.0 0.0" />
   </joint>
-  <joint name="table_to_wobj_reference" type="fixed">
+  <!-- <joint name="table_to_wobj_reference" type="fixed">
     <parent link="table" />
     <child link = "wobj_reference" />
     <origin xyz="0.5 0.0 -0.055" rpy="0.0 0.0 0.0" />
-  </joint>
-  <joint name="wobj_reference_to_wobj" type="fixed">
+  </joint> -->
+  <!-- <joint name="wobj_reference_to_wobj" type="fixed">
     <parent link="wobj_reference" />
     <child link = "wobj" />
     <origin xyz="0 0.0 0.0" rpy="0.0 0.0 -${90 * pi / 180}" />
-  </joint>
+  </joint> -->
   <joint name="tool0_to_glue_gun" type="fixed">
 		<parent link="tool0"/>

Commit message: fix robot position in urdf

File: gluebot_support/urdf/gluebot.xacro (robot description, xacro)
@@ -73,5 +73,5 @@
     <parent link="table" />
     <child link = "base_link" />
-    <origin xyz="0.0 0.0 0.0" rpy="0.0 0.0 0.0" />
+    <origin xyz="0.0 0.0 0.0" rpy="0.0 0.0 ${-45 * pi / 180}" />
   </joint>
   <!-- <joint name="table_to_wobj_reference" type="fixed">
@@ -88,5 +88,5 @@
 		<parent link="tool0"/>
 		<child link="glue_gun"/>
-		<origin rpy="0 0 0" xyz="0 0 0"/>
+		<origin rpy="0 0 ${-45 * pi / 180}" xyz="0 0 0"/>
 		<axis xyz="0 0 0"/>
 	</joint>

Commit message: fix robot position in urdf
(cherry picked from commit 6f2bfb5367791141646325a25c3c64974ca11201)

File: gluebot_support/urdf/gluebot.xacro (robot description, xacro)
@@ -67,5 +67,5 @@
     <parent link="table" />
     <child link = "base_link" />
-    <origin xyz="0.0 0.0 0.0" rpy="0.0 0.0 0.0" />
+    <origin xyz="0.0 0.0 0.0" rpy="0.0 0.0 ${-45 * pi / 180}" />
   </joint>
   <joint name="table_to_wobj_reference" type="fixed">
@@ -82,5 +82,5 @@
 		<parent link="tool0"/>
 		<child link="glue_gun"/>
-		<origin rpy="0 0 0" xyz="0 0 0"/>
+		<origin rpy="0 0 ${-45 * pi / 180}" xyz="0 0 0"/>
 		<axis xyz="0 0 0"/>
 	</joint>

Commit message: add circle task

File: gluebot_support/urdf/gluebot.xacro (robot description, xacro)
@@ -64,4 +64,5 @@
 		  </collision>
   </link>
+  <link name="glue_gun_tip"/>
   <link name="tool_tip"/>
   <joint name="world_to_table" type="fixed">
@@ -91,9 +92,15 @@
 		<axis xyz="0 0 0"/>
 	</joint>
-	<joint name="glue_gun_to_tool_tip" type="fixed">
+  <joint name="glue_gun_to_glue_tip" type="fixed">
 		<parent link="glue_gun"/>
-		<child link="tool_tip"/>
+		<child link="glue_gun_tip"/>
 		<origin rpy="0 ${45 * pi / 180} 0" xyz="0.009664 0 0.272478"/>
 		<axis xyz="0 0 0"/>
 	</joint>
+	<joint name="glue_tip_to_tool_tip" type="fixed">
+		<parent link="glue_gun_tip"/>
+		<child link="tool_tip"/>
+		<origin rpy="0 0 0" xyz="0 0 0.005"/>
+		<axis xyz="0 0 0"/>
+	</joint>
 </robot>

Commit message: new tool tip dimensions

File: gluebot_support/urdf/gluebot.xacro (robot description, xacro)
@@ -92,8 +92,9 @@
 		<axis xyz="0 0 0"/>
 	</joint>
+<!-- <origin rpy="0 ${45 * pi / 180} 0" xyz="0.009664 0 0.272478"/> -->
   <joint name="glue_gun_to_glue_tip" type="fixed">
 		<parent link="glue_gun"/>
 		<child link="glue_gun_tip"/>
-		<origin rpy="0 ${45 * pi / 180} 0" xyz="0.009664 0 0.272478"/>
+		<origin rpy="0 ${45 * pi / 180} 0" xyz="0.01015 0 0.3109"/>
 		<axis xyz="0 0 0"/>
 	</joint>

Commit message: add new workcell model

File: gluebot_support/urdf/gluebot.xacro (robot description, xacro)
@@ -21,5 +21,5 @@
     <origin xyz="-0.25 -0.5 1.25" rpy="0 3.14159 0"/>
   </joint>
-  <link name="table">
+  <!-- <link name="table">
     <visual>
       <geometry>
@@ -34,4 +34,32 @@
 			<origin rpy="0 0 0" xyz="0 0 0"/>
 		  </collision>
+  </link> -->
+  <link name="frame">
+    <visual>
+      <geometry>
+        <mesh filename="package://gluebot_support/meshes/workcell_ur5_simple.stl"/>
+      </geometry>
+		<origin rpy="0 0 0" xyz="0 0 0"/>
+    </visual>
+		<collision>
+		    <geometry>
+		      <mesh filename="package://gluebot_support/meshes/workcell_ur5_simple.stl"/>
+		    </geometry>
+			<origin rpy="0 0 0" xyz="0 0 0"/>
+		  </collision>
+  </link>
+  <link name="table">
+    <visual>
+      <geometry>
+        <box size="0.75 1.2 0.05"/>
+      </geometry>
+		  <origin rpy="0 0 0" xyz="0 0 0"/>
+    </visual>
+		<collision>
+		    <geometry>
+		      <box size="0.75 1.2 0.05"/>>
+		    </geometry>
+			  <origin rpy="0 0 0" xyz="0 0 0"/>
+		</collision>
   </link>
   <!-- <link name="wobj_reference"/> -->
@@ -66,11 +94,16 @@
   <link name="glue_gun_tip"/>
   <link name="tool_tip"/>
-  <joint name="world_to_table" type="fixed">
+  <joint name="world_to_frame" type="fixed">
+    <parent link="world" />
+    <child link = "frame" />
+    <origin xyz="0.0 0.0 0.0" rpy="0.0 0.0 0.0" />
+  </joint>
+   <joint name="world_to_table" type="fixed">
     <parent link="world" />
     <child link = "table" />
-    <origin xyz="0.0 0.0 0.0" rpy="0.0 0.0 0.0" />
+    <origin xyz="${0.245 + 0.75/2} -0.15 ${-0.05 / 2 - 0.16715}" rpy="0 0 0" />
   </joint>
-  <joint name="table_to_base_link" type="fixed">
-    <parent link="table" />
+  <joint name="world_to_base_link" type="fixed">
+    <parent link="world" />
     <child link = "base_link" />
     <origin xyz="0.0 0.0 0.0" rpy="0.0 0.0 ${-45 * pi / 180}" />

Commit message: update urdf

File: gluebot_support/urdf/gluebot.xacro (robot description, xacro)
@@ -14,4 +14,13 @@
     wrist_3_lower_limit="${-pi}" wrist_3_upper_limit="${pi}"
   />
+  <material name="blue">
+    <color rgba="0 0 0.8 1"/>
+  </material>
+  <material name="grey">
+    <color rgba="0.8 0.8 0.8 1"/>
+  </material>
+  <material name="white">
+    <color rgba="1 1 1 1"/>
+  </material>
   <link name="world" />
   <link name="camera_frame"/>
@@ -41,4 +50,5 @@
       </geometry>
 		<origin rpy="0 0 0" xyz="0 0 0"/>
+    <material name="grey"/>
     </visual>
 		<collision>
@@ -55,8 +65,39 @@
       </geometry>
 		  <origin rpy="0 0 0" xyz="0 0 0"/>
+      <material name="white"/>
     </visual>
 		<collision>
 		    <geometry>
 		      <box size="0.75 1.2 0.05"/>>
+		    </geometry>
+			  <origin rpy="0 0 0" xyz="0 0 0"/>
+		</collision>
+  </link>
+  <link name="camera_protection">
+    <visual>
+      <geometry>
+        <box size="0.2 0.35 0.2"/>
+      </geometry>
+		  <origin rpy="0 0 0" xyz="0 0 0"/>
+      <material name="grey"/>
+    </visual>
+		<collision>
+		    <geometry>
+		      <box size="0.2 0.35 0.2"/>>
+		    </geometry>
+			  <origin rpy="0 0 0" xyz="0 0 0"/>
+		</collision>
+  </link>
+  <link name="back_wall">
+    <visual>
+      <geometry>
+        <box size="0.1 2.0 2.0"/>
+      </geometry>
+		  <origin rpy="0 0 0" xyz="0 0 0"/>
+      <material name="blue"/>
+    </visual>
+		<collision>
+		    <geometry>
+		      <box size="0.1 2.0 2.0"/>>
 		    </geometry>
 			  <origin rpy="0 0 0" xyz="0 0 0"/>
@@ -104,4 +145,14 @@
     <origin xyz="${0.245 + 0.75/2} -0.15 ${-0.05 / 2 - 0.16715}" rpy="0 0 0" />
   </joint>
+  <joint name="world_to_camera_protection" type="fixed">
+    <parent link="world" />
+    <child link = "camera_protection" />
+    <origin xyz="0.625 -0.195 0.872" rpy="0 0 0" />
+  </joint>
+   <joint name="world_to_back_wall" type="fixed">
+    <parent link="world" />
+    <child link = "back_wall" />
+    <origin xyz="-0.295 -0.195 ${-0.173 + 1}" rpy="0 0 0" />
+  </joint>
   <joint name="world_to_base_link" type="fixed">
     <parent link="world" />

Commit message: fix tool model

File: gluebot_support/urdf/gluebot.xacro (robot description, xacro)
@@ -122,13 +122,13 @@
     <visual>
       <geometry>
-        <mesh filename="package://gluebot_support/meshes/visual/GlueBot4.stl" scale="0.01 0.01 0.01"/>
+        <mesh filename="package://gluebot_support/meshes/tool.stl" scale="0.001 0.001 0.001"/>
       </geometry>
-		<origin rpy="0 0 0" xyz="0.043 0.043 0"/>
+		<origin rpy="0 0 0" xyz="0.044 -0.044 0.0141"/>
     </visual>
 		<collision>
 		    <geometry>
-		      <mesh filename="package://gluebot_support/meshes/collision/GlueBot4.stl" scale="0.01 0.01 0.01"/>
+		      <mesh filename="package://gluebot_support/meshes/tool.stl" scale="0.001 0.001 0.001"/>
 		    </geometry>
-			<origin rpy="0 0 0" xyz="0.043 0.043 0"/>
+			<origin rpy="0 0 0" xyz="0.044 -0.044 0.0141"/>
 		  </collision>
   </link>

Commit message: set table hight

File: gluebot_support/urdf/gluebot.xacro (robot description, xacro)
@@ -143,5 +143,5 @@
     <parent link="world" />
     <child link = "table" />
-    <origin xyz="${0.245 + 0.75/2} -0.15 ${-0.05 / 2 - 0.16715}" rpy="0 0 0" />
+    <origin xyz="${0.245 + 0.75/2} -0.15 ${-0.05 / 2 - 0.140}" rpy="0 0 0" />
   </joint>
   <joint name="world_to_camera_protection" type="fixed">

Commit message: update gluebot.xacro dimensions

File: gluebot_support/urdf/gluebot.xacro (robot description, xacro)
@@ -24,9 +24,9 @@
   </material>
   <link name="world" />
-  <link name="camera_frame"/>
+  <link name="camera"/>
   <joint name="world_to_camera" type="fixed">
     <parent link="world"/>
-    <child link="camera_frame"/>
-    <origin xyz="-0.25 -0.5 1.25" rpy="0 3.14159 0"/>
+    <child link="camera"/>
+    <origin xyz="0.625 -0.195 0.872" rpy="0 ${pi} ${pi / 2}"/>
   </joint>
   <!-- <link name="table">
